File: PCB/BuckDevel/BuckDevel.sch (KiCad schematic (older format))
At the start: 27 parts

Commit message: Bass hit analysis
I did an analysis of how bass hits will affect the power rails
Parts:
- added C?: EKMM451VSN391MA40S (470uF, 450V), SamacSys_Parts:EKMM451VSN391MA40S, symbol Device:CP1
- added C? (x6): 1uF, 25V, X5R, Capacitors_SMD:C_0402, symbol Device:C
- added C? (x3): 2.2uF, 25V, X5R, Capacitors_SMD:C_0402, symbol Device:C
- added C? (x6): 100n, 16V, X7R, Capacitors_SMD:C_0402, symbol Device:C
- added C? (x12): 100nF, 630V, X7R, Capacitors_SMD:C_1812, symbol Device:C
- added C? (x3): ALC70C332FP350, ALC70C332FP350, symbol SamacSys_Parts:ALC70C332FP350
- added D? (x6): MSS1P2L, SamacSys_Parts:MicroSMP_(DO-219AD), symbol SamacSys_Parts:MSS1P2L
- added D? (x3): GB01SLT06-214, SamacSys_Parts:DO-214AA, symbol SamacSys_Parts:GB01SLT06-214
- added IC? (x3): SI8274GB1-IM1, SI8274GB1IM1, symbol SamacSys_Parts:SI8274GB1-IM1
- added IC? (x3): TPS70960DBVR, SOT95P280X145-5N, symbol SamacSys_Parts:TPS70960DBVR
- added L? (x3): 74437529203471, SamacSys_Parts:74437529203471, symbol SamacSys_Parts:74437529203471
- added Q? (x6): GS-065-011-1-L, GS0650111L, symbol SamacSys_Parts:GS-065-011-1-L
- added R? (x9): 15R, Resistors_SMD:R_0402, symbol Device:R
- added R? (x6): 2R, Resistors_SMD:R_0402, symbol Device:R
- added R? (x6): 10k, Resistors_SMD:R_0402, symbol Device:R
Connections:
- net +12V: now also C?.1, C?.1, C?.1, D?.2 (A), D?.2 (A), D?.2 (A)
- net +3V3: now also C?.1, C?.1, C?.1, IC?.7 (VDDI), IC?.7 (VDDI), IC?.7 (VDDI)
- net 6V_LS: now also C?.1, C?.1, C?.1, IC?.10 (VDDB), IC?.10 (VDDB), IC?.10 (VDDB)
- net EN_GD: now also IC?.5 (EN), IC?.5 (EN), IC?.5 (EN)
- net GND: now also C?.2, C?.2, C?.2, C?.2, C?.2, C?.2, C?.2, C?.2, C?.2, C?.2, C?.2, C?.2, C?.2, C?.2, C?.2, C?.2, C?.2, C?.2, C?.2, C?.2, C?.2, C?.2, C?.2 (-VE), C?.2 (-VE), C?.2 (-VE), IC?.4 (GNDI), IC?.4 (GNDI), IC?.4 (GNDI), IC?.8 (GNDB), IC?.8 (GNDB), IC?.8 (GNDB), Q?.3 (SS), Q?.3 (SS), Q?.3 (SS), Q?.6 (S), Q?.6 (S), Q?.6 (S), R?.1, R?.1, R?.1, R?.2, R?.2, R?.2
- net PWM_0: now also IC?.2 (PWM), IC?.2 (PWM), IC?.2 (PWM)
- net VBUS: now also C?.1, C?.1, C?.1, C?.1, C?.1, C?.1, C?.1, C?.1, C?.1, C?.1, C?.1, C?.1, C?.1, Q?.10 (D_5), Q?.10 (D_5), Q?.10 (D_5), Q?.5 (D_1), Q?.5 (D_1), Q?.5 (D_1), Q?.7 (D_2), Q?.7 (D_2), Q?.7 (D_2), Q?.8 (D_3), Q?.8 (D_3), Q?.8 (D_3), Q?.9 (D_4), Q?.9 (D_4), Q?.9 (D_4)
- new net: IC?.12 (GNDA), Q?.3 (SS), R?.2 (x3)
- new net: Q?.4 (G), R?.1, R?.2, R?.2 (x3)
- new net: L?.1, Q?.10 (D_5), Q?.5 (D_1), Q?.6 (S), Q?.7 (D_2), Q?.8 (D_3), Q?.9 (D_4) (x3)
- new net: D?.1 (K), IC?.13 (VOA), R?.1 (x3)
- new net: C?.1, IC?.14 (VDDA), IC?.5 (OUT) (x3)
- new net: IC?.6 (DT), R?.1 (x3)
- new net: D?.1 (K), IC?.9 (VOB), R?.1 (x3)
- new net: Q?.4 (G), R?.2, R?.2, R?.2 (x3)
- new net: D?.2 (A), R?.1 (x6)
- new net: C?.1, D?.1 (K), IC?.1 (IN) (x3)
- new net: C?.2, C?.2, IC?.2 (GND) (x3)
- new net P1: L?.2
- new net P2: L?.2
- new net P3: L?.2
- new net PWR_OUT: C?.1 (+VE), C?.1 (+VE), C?.1 (+VE)
- no-connect marks 10 -> 43
Other:
- note added: "Current and voltage sensors"
- note added: "Isolation"
- note added: "MCU sheet"
- note added: "connector"
- note removed: "Bulk storage capacitor (450V rating 390uF)"
- moved on the sheet: C?, D?, IC?, L?, Q?, R?

Commit message: pending updates mostly mcu schematic
Parts:
- removed C? (x2): 1uF, 25V, X5R, Capacitors_SMD:C_0402, symbol Device:C
- removed C?: 2.2uF, 25V, X5R, Capacitors_SMD:C_0402, symbol Device:C
- removed C? (x2): 100n, 16V, X7R, Capacitors_SMD:C_0402, symbol Device:C
- removed C? (x4): 100nF, 630V, X7R, Capacitors_SMD:C_1812, symbol Device:C
- removed D? (x2): MSS1P2L, SamacSys_Parts:MicroSMP_(DO-219AD), symbol SamacSys_Parts:MSS1P2L
- removed D?: GB01SLT06-214, SamacSys_Parts:DO-214AA, symbol SamacSys_Parts:GB01SLT06-214
- removed IC?: SI8274GB1-IM1, SI8274GB1IM1, symbol SamacSys_Parts:SI8274GB1-IM1
- removed IC?: TPS70960DBVR, SOT95P280X145-5N, symbol SamacSys_Parts:TPS70960DBVR
- removed L? (x4): 74437529203471, SamacSys_Parts:74437529203471, symbol SamacSys_Parts:74437529203471
- removed Q? (x7): GS-065-011-1-L, GS0650111L, symbol SamacSys_Parts:GS-065-011-1-L
- removed R? (x3): 15R, Resistors_SMD:R_0402, symbol Device:R
- removed R? (x2): 2R, Resistors_SMD:R_0402, symbol Device:R
- removed R? (x2): 10k, Resistors_SMD:R_0402, symbol Device:R
- added C? (x3): 100n, 16V, X7R, Capacitors_SMD:C_0402, symbol Device:C
- added L? (x3): 74437529203221, 74437529203221, symbol SamacSys_Parts:74437529203221
- added Q? (x5): GS-065-011-1-L, SamacSys_Parts:GS0650111L_Therm, symbol SamacSys_Parts:GS-065-011-1-L
- Q?: footprint GS0650111L -> SamacSys_Parts:GS0650111L_Therm
Connections:
- net GND: now also Q?.3 (SS), Q?.3 (SS), Q?.3 (SS), Q?.6 (S), Q?.6 (S), Q?.6 (S)
- net P0: now also L?.2
- net P1: now also L?.2
- net P2: now also L?.2
- net PWM_0: no longer IC?.2 (PWM), IC?.2 (PWM)
- net VBUS: now also Q?.10 (D_5), Q?.10 (D_5), Q?.5 (D_1), Q?.5 (D_1), Q?.7 (D_2), Q?.7 (D_2), Q?.8 (D_3), Q?.8 (D_3), Q?.9 (D_4), Q?.9 (D_4)
- net at Q?.6 (S): now also L?.1, Q?.10 (D_5), Q?.5 (D_1), Q?.7 (D_2), Q?.8 (D_3), Q?.9 (D_4)
- net at R?.2, R?.2, R?.2: now also Q?.4 (G) (x3)
- net at C?.1, IC?.14 (VDDA), IC?.5 (OUT): now also C?.1 (x3)
- net at C?.2, C?.2, IC?.2 (GND): now also C?.2 (x3)
- net at IC?.12 (GNDA), R?.2: now also Q?.3 (SS) (x2)
- net at R?.1, R?.2, R?.2: now also Q?.4 (G) (x2)
- net PWR_OUT renamed ISENSE/PWR_OUT
- new net: L?.1, Q?.10 (D_5), Q?.5 (D_1), Q?.6 (S), Q?.7 (D_2), Q?.8 (D_3), Q?.9 (D_4) (x2)
- new net PWM_1: IC?.2 (PWM)
- new net PWM_2: IC?.2 (PWM)
- no-connect marks 43 -> 34
Other:
- note added: "220uH"
- note added: "2oZ copper required for heat spreading, 1mm thick PCB\n"
- note added: "300V, 12A Bus"
- note added: "ADC range?"
- note added: "Converter switched at 9*48kHz = 432 kHz. Nominal Vout = 300V, current limit at 3*4A=12A"
- note added: "Total = 9900uF"
- note added: "Vbus = 390V from PFC stage"
- note removed: "2oZ copper required for heat spreading\n"
- note removed: "470uH"
- moved on the sheet: C?
